Commit message: feat : add gazebo-rviz screenshot

File: mastering_ros_robot_description_pkg/urdf/pan_tilt_generated2.urdf (robot description, URDF)
Before this commit: robot pan_tilt, 3 links, 2 joints
Links:
- link tilt_link: geometry collision cylinder length=0.4 radius=0.24000000000000002; visual cylinder length=0.4 radius=0.04

File: mastering_ros_robot_description_pkg/urdf/seven_dof_arm.xacro (robot description, xacro)
@@ -58,14 +58,13 @@
    </xacro:macro>
    <xacro:macro name="transmission_block" params="joint_name">
-	  <transmission name="tran1">
-	    <type>transmission_interface/SimpleTransmission</type>
-	    <joint name="${joint_name}">
-	      <hardwareInterface>hardware_interface/PositionJointInterface</hardwareInterface>
-	    </joint>
-	    <actuator name="motor1">
-	      <hardwareInterface>hardware_interface/PositionJointInterface</hardwareInterface>
-	      <mechanicalReduction>1</mechanicalReduction>
-	    </actuator>
-	  </transmission>
+    <transmission name="trans_${joint_name}">
+      <type>transmission_interface/SimpleTransmission</type>
+        <joint name="${joint_name}">
+            <hardwareInterface>hardware_interface/PositionJointInterface</hardwareInterface>
+        </joint>
+        <actuator name="motor_${joint_name}"> <hardwareInterface>hardware_interface/PositionJointInterface</hardwareInterface>
+            <mechanicalReduction>1</mechanicalReduction>
+        </actuator>
+    </transmission>
    </xacro:macro>
 <!-- BOTTOM FIXED LINK
